Commit message: Added Camera to Jackal

File: jackal_foxy/jackal-foxy-devel/jackal_description/urdf/accessories.urdf.xacro (robot description, xacro)
@@ -202,4 +202,5 @@
   <!--xacro:include filename="$(find pointgrey_camera_description)/urdf/pointgrey_flea3.urdf.xacro" /-->
   <!-- If enabled, generate the flea3 camera payload with a tilt of 30 degrees. -->
+  <!-- -->
   <xacro:if value="$(optenv JACKAL_FLEA3 0)">
     <xacro:property name="name" value="$(optenv JACKAL_FLEA3_NAME front)" />
@@ -209,8 +210,9 @@
     <xacro:property name="prefix" value="$(optenv JACKAL_FLEA3_PREFIX ${mount})" />
     <xacro:property name="parent" value="$(optenv JACKAL_FLEA3_PARENT ${mount}_mount)" />
-    <xacro:pointgrey_flea3 frame="${prefix}_camera" name="${name}"
+    <!-- <xacro:pointgrey_flea3 frame="${prefix}_camera" name="${name}"
       camera_x="0.0754" camera_y="0.029" camera_z="0.029"
-      camera_mass="0.085" hfov="1.0471975512" fps="60" width="640" height="512"/>
+      camera_mass="0.085" hfov="1.0471975512" fps="60" width="640" height="512"/> -->
     <!-- Mount Enabled -->
+    <!--  -->
     <xacro:if value="${tower}">
       <xacro:camera_mount prefix="${prefix}" tilt="${tilt}"/>

File: jackal_foxy/jackal-foxy-devel/jackal_description/urdf/accessories/camera_mount.urdf.xacro (robot description, xacro)
@@ -19,4 +19,31 @@
       </visual>
     </link>
+    <!-- camera -->
+      <gazebo reference="${prefix}_camera_beam">
+        <sensor type="camera" name="${prefix}_camera_beam">
+          <update_rate> 30.0 </update_rate>
+          <always_on> 1 </always_on>
+          <topic> image </topic>
+          <camera name="tool">
+            <horizontal_fov> 1.0 </horizontal_fov>
+            <image>
+              <width> 800 </width>
+              <height> 800 </height>
+              <format>R8G8B8</format>
+            </image>
+            <clip>
+              <near> 0.02 </near>
+              <far> 300 </far>
+            </clip>
+            <noise>
+              <mean> 0.0 </mean>
+              <stddev> 0.01 </stddev>
+            </noise>
+          </camera>
+          <plugin filename="ignition-gazebo-sensors-system"
+            name="ignition::gazebo::systems::Sensors">
+          </plugin>
+        </sensor>
+      </gazebo>
     <joint name="${prefix}_camera_pivot_joint" type="fixed">
       <origin xyz="0.102 0 0.008" rpy="0 ${tilt} 0" />

File: jackal_foxy/jackal-foxy-devel/jackal_description/urdf/accessories/hokuyo_ust10.urdf.xacro (robot description, xacro)
@@ -13,4 +13,10 @@
         </inertial>
       </link>
+      <!-- <link name="${frame}_camera"> </link>
+      <joint name="${frame}_joint" type="fixed">
+        <origin xyz="0 0 0" rpy="0 0 0" />
+        <parent link="${frame}"/>
+        <child link="${frame}_camera" />
+      </joint> -->
       <!-- <gazebo reference="${frame}">
         <turnGravityOff>true</turnGravityOff>
@@ -50,35 +56,62 @@
       </gazebo> -->
       <gazebo reference="${frame}">
-            <sensor type="gpu_lidar" name="${frame}">
-                <ignition_frame_id>${frame}</ignition_frame_id>
-                <update_rate> 40.00 </update_rate>
-                <always_on> 1 </always_on>
-                <topic> range </topic>
-                <ray>
-                    <scan>
-                        <horizontal>
-                            <samples>${sample_size}</samples>
-                            <resolution>1</resolution>
-                            <min_angle>${min_angle}</min_angle>
-                            <max_angle>${max_angle}</max_angle>
-                        </horizontal>
-                        <vertical>
-                            <samples>5</samples>
-                            <resolution>1</resolution>
-                            <min_angle> -.2616</min_angle>
-                            <max_angle> .2616</max_angle>
-                        </vertical>
-                    </scan>
-                    <range>
-                        <min>${min_range}</min>
-                        <max>${max_range}</max>
-                        <resolution>0.01</resolution>
-                    </range>
-                </ray>
-                <plugin filename="ignition-gazebo-sensors-system"
-                    name="ignition::gazebo::systems::Sensors">
-                </plugin>
-            </sensor>
-        </gazebo>
+        <sensor type="gpu_lidar" name="${frame}">
+          <ignition_frame_id>${frame}</ignition_frame_id>
+          <update_rate> 40.00 </update_rate>
+          <always_on> 1 </always_on>
+          <topic> range </topic>
+          <ray>
+            <scan>
+              <horizontal>
+                <samples>${sample_size}</samples>
+                <resolution>1</resolution>
+                <min_angle>${min_angle}</min_angle>
+                <max_angle>${max_angle}</max_angle>
+              </horizontal>
+              <vertical>
+                <samples>5</samples>
+                <resolution>1</resolution>
+                <min_angle> -.2616</min_angle>
+                <max_angle> .2616</max_angle>
+              </vertical>
+            </scan>
+            <range>
+              <min>${min_range}</min>
+              <max>${max_range}</max>
+              <resolution>0.01</resolution>
+            </range>
+          </ray>
+          <plugin filename="ignition-gazebo-sensors-system"
+                  name="ignition::gazebo::systems::Sensors">
+          </plugin>
+        </sensor>
+      </gazebo>
+              <!-- camera -->
+      <gazebo reference="${frame}">
+        <sensor type="camera" name="${frame}_camera">
+          <update_rate> 30.0 </update_rate>
+          <always_on> 1 </always_on>
+          <topic> image </topic>
+          <camera name="tool">
+            <horizontal_fov> 1.0 </horizontal_fov>
+            <image>
+              <width> 800 </width>
+              <height> 800 </height>
+              <format>R8G8B8</format>
+            </image>
+            <clip>
+              <near> 0.02 </near>
+              <far> 300 </far>
+            </clip>
+            <noise>
+              <mean> 0.0 </mean>
+              <stddev> 0.01 </stddev>
+            </noise>
+          </camera>
+          <!-- <plugin filename="ignition-gazebo-sensors-system"
+            name="ignition::gazebo::systems::Sensors">
+          </plugin> -->
+        </sensor>
+      </gazebo>
     </xacro:macro>
     <xacro:hokuyo_ust10 frame="${prefix}_laser" topic="${topic}"/>
